File: INA138_sen/INA138_sen.sch (KiCad schematic (older format))
At the start: 18 parts, among them J1 Screw_Terminal_01x02, J2 Screw_Terminal_01x02, J3 Screw_Terminal_01x02, U1 INA138

Commit message: changed footprint of INA138
Parts:
- U1: footprint Package_TO_SOT_SMD:SOT-223-5 -> Package_TO_SOT_SMD:SOT-23-5
Changed lines of the file:
@@
 EESchema Schematic File Version 4
+LIBS:INA138_sen-cache
 EELAYER 26 0
 EELAYER END
@@
 F 0 "U1" V 4954 2159 50  0000 R CNN
 F 1 "INA138" V 5045 2159 50  0000 R CNN
-F 2 "Package_TO_SOT_SMD:SOT-223-5" H 5000 2500 50  0001 C CNN
+F 2 "Package_TO_SOT_SMD:SOT-23-5" H 5000 2500 50  0001 C CNN
 F 3 "http://www.ti.com/lit/ds/symlink/ina138.pdf" H 5000 2505 50  0001 C CNN
 	1    5000 2500
@@
 Wire Wire Line
 	5450 3000 5350 3000
-Wire Wire Line
-	5300 2400 5450 2400
-Wire Wire Line
-	5450 2400 5450 2850
-Connection ~ 5450 2850
 $Comp
 L power:GND #PWR08
@@
 	1    0    0    -1
 $EndComp
-Connection ~ 5450 3000
 $Comp
 L power:GND #PWR02
@@
 Wire Wire Line
 	3800 2500 3800 2550
-Wire Wire Line
-	5450 3000 5450 3350
 $Comp
 L power:VCC #PWR01
@@
 	5500 1150 5200 1150
 Connection ~ 5200 1150
+Wire Wire Line
+	5300 2400 5450 2400
+Wire Wire Line
+	5450 2400 5450 2850
+Connection ~ 5450 2850
+Wire Wire Line
+	5450 3000 5450 3150
+Connection ~ 5450 3000
 $EndSCHEMATC

Commit message: Completed PCB layout
Parts:
- added J4: Conn_01x02_Female, Connector_PinHeader_2.54mm:PinHeader_1x02_P2.54mm_Vertical, symbol Connector:Conn_01x02_Female
Connections:
- net labels added: I+, I-, VOUT
- wire segments 63 -> 71
